Commit message: removed abs paths, now allowing parsin URDF and specifying mesh root dir and, optionally, subdirs

File: tests/files/centauro.urdf (robot description, URDF)
Before this commit: robot centauro, 57 links, 56 joints
Links:
- added link world
- link D435_head_camera_link: geometry collision box size=0.02505 0.09 0.025; visual mesh filename=meshes/realsense/d435.dae
- link D435i_camera_link: geometry collision box size=0.02505 0.09 0.025; visual mesh filename=meshes/realsense/d435.dae
- link ankle1_1: geometry collision mesh filename=meshes/v2/collision/ankle-pitch.stl scale=0.001 0.001 -0.001; visual mesh filename=meshes/v2/ankle-pitch.stl scale=0.001 0.001 -0.001
- link ankle1_2: geometry collision mesh filename=meshes/v2/collision/ankle-pitch.stl scale=0.001 0.001 0.001; visual mesh filename=meshes/v2/ankle-pitch.stl scale=0.001 0.001 0.001
- link ankle1_3: geometry collision mesh filename=meshes/v2/collision/ankle-pitch.stl scale=0.001 0.001 -0.001; visual mesh filename=meshes/v2/ankle-pitch.stl scale=0.001 0.001 -0.001
- link ankle1_4: geometry collision mesh filename=meshes/v2/collision/ankle-pitch.stl scale=0.001 0.001 0.001; visual mesh filename=meshes/v2/ankle-pitch.stl scale=0.001 0.001 0.001
- link ankle2_1: geometry collision mesh filename=meshes/v2/collision/mesh_ankle-yaw_wheel23.stl scale=0.001 -0.001 0.001; visual mesh filename=meshes/v2/mesh_ankle-yaw_wheel23.stl scale=0.001 -0.001 0.001
- link ankle2_2: geometry collision mesh filename=meshes/v2/collision/mesh_ankle-yaw_wheel23.stl scale=0.001 0.001 0.001; visual mesh filename=meshes/v2/mesh_ankle-yaw_wheel23.stl scale=0.001 0.001 0.001
- link ankle2_3: geometry collision mesh filename=meshes/v2/collision/mesh_ankle-yaw_wheel23.stl scale=0.001 -0.001 0.001; visual mesh filename=meshes/v2/mesh_ankle-yaw_wheel23.stl scale=0.001 -0.001 0.001
- link ankle2_4: geometry collision mesh filename=meshes/v2/collision/mesh_ankle-yaw_wheel23.stl scale=0.001 0.001 0.001; visual mesh filename=meshes/v2/mesh_ankle-yaw_wheel23.stl scale=0.001 0.001 0.001
- link arm1_1: geometry collision mesh filename=meshes/simple/ShoulderPitch.STL scale=0.001 -0.001 0.001; visual mesh filename=meshes/ShoulderPitch.STL scale=0.001 -0.001 0.001
- link arm1_2: geometry collision mesh filename=meshes/simple/ShoulderRoll.STL scale=0.001 -0.001 0.001; visual mesh filename=meshes/ShoulderRoll.STL scale=0.001 -0.001 0.001
- link arm1_3: geometry collision mesh filename=meshes/simple/ShoulderYaw.STL scale=0.001 -0.001 0.001; visual mesh filename=meshes/ShoulderYaw.STL scale=0.001 -0.001 0.001
- link arm1_4: geometry collision mesh filename=meshes/simple/Elbow.STL scale=0.001 -0.001 0.001; visual mesh filename=meshes/Elbow.STL scale=0.001 -0.001 0.001
- link arm1_5: geometry collision mesh filename=meshes/simple/Forearm.STL scale=0.001 -0.001 0.001; visual mesh filename=meshes/Forearm.STL scale=0.001 -0.001 0.001
- link arm1_6: geometry collision mesh filename=meshes/simple/wrist_pitch_right.stl scale=0.001 -0.001 0.001; visual mesh filename=meshes/wrist_pitch_right.stl scale=0.001 -0.001 0.001
- link arm2_1: geometry collision mesh filename=meshes/simple/ShoulderPitch.STL scale=0.001 0.001 0.001; visual mesh filename=meshes/ShoulderPitch.STL scale=0.001 0.001 0.001
- link arm2_2: geometry collision mesh filename=meshes/simple/ShoulderRoll.STL scale=0.001 0.001 0.001; visual mesh filename=meshes/ShoulderRoll.STL scale=0.001 0.001 0.001
- link arm2_3: geometry collision mesh filename=meshes/simple/ShoulderYaw.STL scale=0.001 0.001 0.001; visual mesh filename=meshes/ShoulderYaw.STL scale=0.001 0.001 0.001
- link arm2_4: geometry collision mesh filename=meshes/simple/Elbow.STL scale=0.001 0.001 0.001; visual mesh filename=meshes/Elbow.STL scale=0.001 0.001 0.001
- link arm2_5: geometry collision mesh filename=meshes/simple/Forearm.STL scale=0.001 0.001 0.001; visual mesh filename=meshes/Forearm.STL scale=0.001 0.001 0.001
- link arm2_6: geometry collision mesh filename=meshes/simple/wrist_pitch_right.stl scale=0.001 0.001 0.001; visual mesh filename=meshes/wrist_pitch_right.stl scale=0.001 0.001 0.001
- link ball1: geometry collision mesh filename=meshes/simple/BallHand.stl scale=0.001 0.001 0.001; visual mesh filename=meshes/BallHand.stl scale=0.001 0.001 0.001
- link ball2: geometry collision mesh filename=meshes/simple/BallHand.stl scale=0.001 0.001 0.001; visual mesh filename=meshes/BallHand.stl scale=0.001 0.001 0.001
- link d435_head_motor: geometry collision mesh filename=meshes/simple/neck-pitch_mesh.stl scale=0.001 0.001 0.001; visual mesh filename=meshes/neck-pitch_mesh.stl scale=0.001 0.001 0.001
- link hip1_1: geometry collision mesh filename=meshes/v2/collision/hip-yaw.stl scale=0.001 -0.001 0.001; visual mesh filename=meshes/v2/hip-yaw.stl scale=0.001 -0.001 0.001
- link hip1_2: geometry collision mesh filename=meshes/v2/collision/hip-yaw.stl scale=0.001 0.001 0.001; visual mesh filename=meshes/v2/hip-yaw.stl scale=0.001 0.001 0.001
- link hip1_3: geometry collision mesh filename=meshes/v2/collision/hip-yaw.stl scale=0.001 -0.001 0.001; visual mesh filename=meshes/v2/hip-yaw.stl scale=0.001 -0.001 0.001
- link hip1_4: geometry collision mesh filename=meshes/v2/collision/hip-yaw.stl scale=0.001 0.001 0.001; visual mesh filename=meshes/v2/hip-yaw.stl scale=0.001 0.001 0.001
- link hip2_1: geometry collision mesh filename=meshes/v2/collision/hip-pitch.stl scale=0.001 0.001 -0.001; visual mesh filename=meshes/v2/hip-pitch.stl scale=0.001 0.001 -0.001
- link hip2_2: geometry collision mesh filename=meshes/v2/collision/hip-pitch.stl scale=0.001 0.001 0.001; visual mesh filename=meshes/v2/hip-pitch.stl scale=0.001 0.001 0.001
- link hip2_3: geometry collision mesh filename=meshes/v2/collision/hip-pitch.stl scale=0.001 0.001 -0.001; visual mesh filename=meshes/v2/hip-pitch.stl scale=0.001 0.001 -0.001
- link hip2_4: geometry collision mesh filename=meshes/v2/collision/hip-pitch.stl scale=0.001 0.001 0.001; visual mesh filename=meshes/v2/hip-pitch.stl scale=0.001 0.001 0.001
- link knee_1: geometry collision mesh filename=meshes/v2/collision/knee.stl scale=0.001 0.001 -0.001; visual mesh filename=meshes/v2/knee.stl scale=0.001 0.001 -0.001
- link knee_2: geometry collision mesh filename=meshes/v2/collision/knee.stl scale=0.001 0.001 0.001; visual mesh filename=meshes/v2/knee.stl scale=0.001 0.001 0.001
- link knee_3: geometry collision mesh filename=meshes/v2/collision/knee.stl scale=0.001 0.001 -0.001; visual mesh filename=meshes/v2/knee.stl scale=0.001 0.001 -0.001
- link knee_4: geometry collision mesh filename=meshes/v2/collision/knee.stl scale=0.001 0.001 0.001; visual mesh filename=meshes/v2/knee.stl scale=0.001 0.001 0.001
- link neck_1: geometry collision mesh filename=meshes/simple/head-base_mesh.stl scale=0.001 0.001 0.001; visual mesh filename=meshes/head-base_mesh.stl scale=0.001 0.001 0.001
- link pelvis: geometry collision mesh filename=meshes/simple/pelvis.stl scale=0.001 0.001 0.001; visual mesh filename=meshes/v2/pelvis.stl scale=0.001 0.001 0.001
- link torso_2: geometry collision mesh filename=meshes/simple/link1_no_head.stl scale=0.001 0.001 0.001; visual mesh filename=meshes/link1_no_head.stl scale=0.001 0.001 0.001
- link velodyne_motor: geometry collision mesh filename=meshes/simple/lidar_mesh.stl scale=0.001 0.001 0.001; visual mesh filename=meshes/lidar_mesh.stl scale=0.001 0.001 0.001
- link wheel_1: geometry collision mesh filename=meshes/v2/collision/mesh_wheel23.stl scale=0.001 0.001 -0.001; visual mesh filename=meshes/v2/mesh_wheel23.stl scale=0.001 0.001 -0.001
- link wheel_2: geometry collision mesh filename=meshes/v2/collision/mesh_wheel23.stl scale=0.001 0.001 0.001; visual mesh filename=meshes/v2/mesh_wheel23.stl scale=0.001 0.001 0.001
- link wheel_3: geometry collision mesh filename=meshes/v2/collision/mesh_wheel23.stl scale=0.001 0.001 -0.001; visual mesh filename=meshes/v2/mesh_wheel23.stl scale=0.001 0.001 -0.001
- link wheel_4: geometry collision mesh filename=meshes/v2/collision/mesh_wheel23.stl scale=0.001 0.001 0.001; visual mesh filename=meshes/v2/mesh_wheel23.stl scale=0.001 0.001 0.001
Joints:
- added joint reference: type floating, parent world, child base_link

Commit message: Signed-off-by: Andrea Patrizi <andreapatrizi1b6e6@gmail.com>

File: tests/files/centauro.urdf (robot description, URDF)
Before this commit: robot centauro, 58 links, 57 joints
Joints:
- joint reference: origin (none) -> xyz=0 0 1 rpy=0 0 0

Commit message: big commit: starting to add homing parser and setter from SRDF + sites parsing fix + other improvs
Signed-off-by: Andrea Patrizi <andreapatrizi1b6e6@gmail.com>

File: tests/files/centauro.urdf (robot description, URDF)
Before this commit: robot centauro, 58 links, 57 joints
Links:
- link D435_head_camera_link: geometry collision box size=0.02505 0.09 0.025; visual mesh filename=/root/ibrido_ws/src/iit-centauro-ros-pkg/centauro_urdf/mesh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
- link D435i_camera_link: geometry collision box size=0.02505 0.09 0.025; visual mesh filename=/root/ibrido_ws/src/iit-centauro-ros-pkg/centauro_urdf/mesh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
- link ankle1_1: geometry collision mesh filename=/root/ibrido_ws/src/iit-centauro-ros-pkg/centauro_urdf/mesh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 scale=0.001 0.001 -0.001; visual mesh filename=/root/ibrido_ws/src/iit-centauro-ros-pkg/centauro_urdf/mesh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 scale=0.001 0.001 -0.001
- link ankle1_2: geometry collision mesh filename=/root/ibrido_ws/src/iit-centauro-ros-pkg/centauro_urdf/mesh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 scale=0.001 0.001 0.001; visual mesh filename=/root/ibrido_ws/src/iit-centauro-ros-pkg/centauro_urdf/mesh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 scale=0.001 0.001 0.001
- link ankle1_3: geometry collision mesh filename=/root/ibrido_ws/src/iit-centauro-ros-pkg/centauro_urdf/mesh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 scale=0.001 0.001 -0.001; visual mesh filename=/root/ibrido_ws/src/iit-centauro-ros-pkg/centauro_urdf/mesh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 scale=0.001 0.001 -0.001
- link ankle1_4: geometry collision mesh filename=/root/ibrido_ws/src/iit-centauro-ros-pkg/centauro_urdf/mesh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 scale=0.001 0.001 0.001; visual mesh filename=/root/ibrido_ws/src/iit-centauro-ros-pkg/centauro_urdf/mesh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 scale=0.001 0.001 0.001
- link ankle2_1: geometry collision mesh filename=/root/ibrido_ws/src/iit-centauro-ros-pkg/centauro_urdf/mesh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 scale=0.001 -0.001 0.001; visual mesh filename=/root/ibrido_ws/src/iit-centauro-ros-pkg/centauro_urdf/mesh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 scale=0.001 -0.001 0.001
- link ankle2_2: geometry collision mesh filename=/root/ibrido_ws/src/iit-centauro-ros-pkg/centauro_urdf/mesh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 scale=0.001 0.001 0.001; visual mesh filename=/root/ibrido_ws/src/iit-centauro-ros-pkg/centauro_urdf/mesh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 scale=0.001 0.001 0.001
- link ankle2_3: geometry collision mesh filename=/root/ibrido_ws/src/iit-centauro-ros-pkg/centauro_urdf/mesh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 scale=0.001 -0.001 0.001; visual mesh filename=/root/ibrido_ws/src/iit-centauro-ros-pkg/centauro_urdf/mesh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 scale=0.001 -0.001 0.001
- link ankle2_4: geometry collision mesh filename=/root/ibrido_ws/src/iit-centauro-ros-pkg/centauro_urdf/mesh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 scale=0.001 0.001 0.001; visual mesh filename=/root/ibrido_ws/src/iit-centauro-ros-pkg/centauro_urdf/mesh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 scale=0.001 0.001 0.001
- link arm1_1: geometry collision mesh filename=/root/ibrido_ws/src/iit-centauro-ros-pkg/centauro_urdf/mesh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 scale=0.001 -0.001 0.001; visual mesh filename=/root/ibrido_ws/src/iit-centauro-ros-pkg/centauro_urdf/mesh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 scale=0.001 -0.001 0.001
- link arm1_2: geometry collision mesh filename=/root/ibrido_ws/src/iit-centauro-ros-pkg/centauro_urdf/mesh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 scale=0.001 -0.001 0.001; visual mesh filename=/root/ibrido_ws/src/iit-centauro-ros-pkg/centauro_urdf/mesh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 scale=0.001 -0.001 0.001
- link arm1_3: geometry collision mesh filename=/root/ibrido_ws/src/iit-centauro-ros-pkg/centauro_urdf/mesh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 scale=0.001 -0.001 0.001; visual mesh filename=/root/ibrido_ws/src/iit-centauro-ros-pkg/centauro_urdf/mesh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 scale=0.001 -0.001 0.001
- link arm1_4: geometry collision mesh filename=/root/ibrido_ws/src/iit-centauro-ros-pkg/centauro_urdf/mesh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 scale=0.001 -0.001 0.001; visual mesh filename=/root/ibrido_ws/src/iit-centauro-ros-pkg/centauro_urdf/mesh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 scale=0.001 -0.001 0.001
- link arm1_5: geometry collision mesh filename=/root/ibrido_ws/src/iit-centauro-ros-pkg/centauro_urdf/mesh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 scale=0.001 -0.001 0.001; visual mesh filename=/root/ibrido_ws/src/iit-centauro-ros-pkg/centauro_urdf/mesh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 scale=0.001 -0.001 0.001
- link arm1_6: geometry collision mesh filename=/root/ibrido_ws/src/iit-centauro-ros-pkg/centauro_urdf/mesh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 scale=0.001 -0.001 0.001; visual mesh filename=/root/ibrido_ws/src/iit-centauro-ros-pkg/centauro_urdf/mesh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 scale=0.001 -0.001 0.001
- link arm2_1: geometry collision mesh filename=/root/ibrido_ws/src/iit-centauro-ros-pkg/centauro_urdf/mesh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 scale=0.001 0.001 0.001; visual mesh filename=/root/ibrido_ws/src/iit-centauro-ros-pkg/centauro_urdf/mesh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 scale=0.001 0.001 0.001
- link arm2_2: geometry collision mesh filename=/root/ibrido_ws/src/iit-centauro-ros-pkg/centauro_urdf/mesh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 scale=0.001 0.001 0.001; visual mesh filename=/root/ibrido_ws/src/iit-centauro-ros-pkg/centauro_urdf/mesh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 scale=0.001 0.001 0.001
- link arm2_3: geometry collision mesh filename=/root/ibrido_ws/src/iit-centauro-ros-pkg/centauro_urdf/mesh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 scale=0.001 0.001 0.001; visual mesh filename=/root/ibrido_ws/src/iit-centauro-ros-pkg/centauro_urdf/mesh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 scale=0.001 0.001 0.001
- link arm2_4: geometry collision mesh filename=/root/ibrido_ws/src/iit-centauro-ros-pkg/centauro_urdf/mesh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 scale=0.001 0.001 0.001; visual mesh filename=/root/ibrido_ws/src/iit-centauro-ros-pkg/centauro_urdf/mesh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 scale=0.001 0.001 0.001
- link arm2_5: geometry collision mesh filename=/root/ibrido_ws/src/iit-centauro-ros-pkg/centauro_urdf/mesh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 scale=0.001 0.001 0.001; visual mesh filename=/root/ibrido_ws/src/iit-centauro-ros-pkg/centauro_urdf/mesh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 scale=0.001 0.001 0.001
- link arm2_6: geometry collision mesh filename=/root/ibrido_ws/src/iit-centauro-ros-pkg/centauro_urdf/mesh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 scale=0.001 0.001 0.001; visual mesh filename=/root/ibrido_ws/src/iit-centauro-ros-pkg/centauro_urdf/mesh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 scale=0.001 0.001 0.001
- link ball1: geometry collision mesh filename=/root/ibrido_ws/src/iit-centauro-ros-pkg/centauro_urdf/mesh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 scale=0.001 0.001 0.001; visual mesh filename=/root/ibrido_ws/src/iit-centauro-ros-pkg/centauro_urdf/mesh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 scale=0.001 0.001 0.001
- link ball2: geometry collision mesh filename=/root/ibrido_ws/src/iit-centauro-ros-pkg/centauro_urdf/mesh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 scale=0.001 0.001 0.001; visual mesh filename=/root/ibrido_ws/src/iit-centauro-ros-pkg/centauro_urdf/mesh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 scale=0.001 0.001 0.001
- link d435_head_motor: geometry collision mesh filename=/root/ibrido_ws/src/iit-centauro-ros-pkg/centauro_urdf/mesh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 scale=0.001 0.001 0.001; visual mesh filename=/root/ibrido_ws/src/iit-centauro-ros-pkg/centauro_urdf/mesh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 scale=0.001 0.001 0.001
- link hip1_1: geometry collision mesh filename=/root/ibrido_ws/src/iit-centauro-ros-pkg/centauro_urdf/mesh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 scale=0.001 -0.001 0.001; visual mesh filename=/root/ibrido_ws/src/iit-centauro-ros-pkg/centauro_urdf/mesh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 scale=0.001 -0.001 0.001
- link hip1_2: geometry collision mesh filename=/root/ibrido_ws/src/iit-centauro-ros-pkg/centauro_urdf/mesh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 scale=0.001 0.001 0.001; visual mesh filename=/root/ibrido_ws/src/iit-centauro-ros-pkg/centauro_urdf/mesh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 scale=0.001 0.001 0.001
- link hip1_3: geometry collision mesh filename=/root/ibrido_ws/src/iit-centauro-ros-pkg/centauro_urdf/mesh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 scale=0.001 -0.001 0.001; visual mesh filename=/root/ibrido_ws/src/iit-centauro-ros-pkg/centauro_urdf/mesh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 scale=0.001 -0.001 0.001
- link hip1_4: geometry collision mesh filename=/root/ibrido_ws/src/iit-centauro-ros-pkg/centauro_urdf/mesh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 scale=0.001 0.001 0.001; visual mesh filename=/root/ibrido_ws/src/iit-centauro-ros-pkg/centauro_urdf/mesh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 scale=0.001 0.001 0.001
- link hip2_1: geometry collision mesh filename=/root/ibrido_ws/src/iit-centauro-ros-pkg/centauro_urdf/mesh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 scale=0.001 0.001 -0.001; visual mesh filename=/root/ibrido_ws/src/iit-centauro-ros-pkg/centauro_urdf/mesh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 scale=0.001 0.001 -0.001
- link hip2_2: geometry collision mesh filename=/root/ibrido_ws/src/iit-centauro-ros-pkg/centauro_urdf/mesh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 scale=0.001 0.001 0.001; visual mesh filename=/root/ibrido_ws/src/iit-centauro-ros-pkg/centauro_urdf/mesh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 scale=0.001 0.001 0.001
- link hip2_3: geometry collision mesh filename=/root/ibrido_ws/src/iit-centauro-ros-pkg/centauro_urdf/mesh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 scale=0.001 0.001 -0.001; visual mesh filename=/root/ibrido_ws/src/iit-centauro-ros-pkg/centauro_urdf/mesh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 scale=0.001 0.001 -0.001
- link hip2_4: geometry collision mesh filename=/root/ibrido_ws/src/iit-centauro-ros-pkg/centauro_urdf/mesh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 scale=0.001 0.001 0.001; visual mesh filename=/root/ibrido_ws/src/iit-centauro-ros-pkg/centauro_urdf/mesh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 scale=0.001 0.001 0.001
- link knee_1: geometry collision mesh filename=/root/ibrido_ws/src/iit-centauro-ros-pkg/centauro_urdf/mesh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 scale=0.001 0.001 -0.001; visual mesh filename=/root/ibrido_ws/src/iit-centauro-ros-pkg/centauro_urdf/mesh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 scale=0.001 0.001 -0.001
- link knee_2: geometry collision mesh filename=/root/ibrido_ws/src/iit-centauro-ros-pkg/centauro_urdf/mesh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 scale=0.001 0.001 0.001; visual mesh filename=/root/ibrido_ws/src/iit-centauro-ros-pkg/centauro_urdf/mesh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 scale=0.001 0.001 0.001
- link knee_3: geometry collision mesh filename=/root/ibrido_ws/src/iit-centauro-ros-pkg/centauro_urdf/mesh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 scale=0.001 0.001 -0.001; visual mesh filename=/root/ibrido_ws/src/iit-centauro-ros-pkg/centauro_urdf/mesh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 scale=0.001 0.001 -0.001
- link knee_4: geometry collision mesh filename=/root/ibrido_ws/src/iit-centauro-ros-pkg/centauro_urdf/mesh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 scale=0.001 0.001 0.001; visual mesh filename=/root/ibrido_ws/src/iit-centauro-ros-pkg/centauro_urdf/mesh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 scale=0.001 0.001 0.001
- link neck_1: geometry collision mesh filename=/root/ibrido_ws/src/iit-centauro-ros-pkg/centauro_urdf/mesh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 scale=0.001 0.001 0.001; visual mesh filename=/root/ibrido_ws/src/iit-centauro-ros-pkg/centauro_urdf/mesh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 scale=0.001 0.001 0.001
- link pelvis: geometry collision mesh filename=/root/ibrido_ws/src/iit-centauro-ros-pkg/centauro_urdf/mesh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 scale=0.001 0.001 0.001; visual mesh filename=/root/ibrido_ws/src/iit-centauro-ros-pkg/centauro_urdf/mesh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 scale=0.001 0.001 0.001
- link torso_2: geometry collision mesh filename=/root/ibrido_ws/src/iit-centauro-ros-pkg/centauro_urdf/mesh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 scale=0.001 0.001 0.001; visual mesh filename=/root/ibrido_ws/src/iit-centauro-ros-pkg/centauro_urdf/mesh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 scale=0.001 0.001 0.001
- link velodyne_motor: geometry collision mesh filename=/root/ibrido_ws/src/iit-centauro-ros-pkg/centauro_urdf/mesh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 scale=0.001 0.001 0.001; visual mesh filename=/root/ibrido_ws/src/iit-centauro-ros-pkg/centauro_urdf/mesh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 scale=0.001 0.001 0.001
- link wheel_1: geometry collision mesh filename=/root/ibrido_ws/src/iit-centauro-ros-pkg/centauro_urdf/mesh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 scale=0.001 0.001 -0.001; visual mesh filename=/root/ibrido_ws/src/iit-centauro-ros-pkg/centauro_urdf/mesh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 scale=0.001 0.001 -0.001
- link wheel_2: geometry collision mesh filename=/root/ibrido_ws/src/iit-centauro-ros-pkg/centauro_urdf/mesh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 scale=0.001 0.001 0.001; visual mesh filename=/root/ibrido_ws/src/iit-centauro-ros-pkg/centauro_urdf/mesh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 scale=0.001 0.001 0.001
- link wheel_3: geometry collision mesh filename=/root/ibrido_ws/src/iit-centauro-ros-pkg/centauro_urdf/mesh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 scale=0.001 0.001 -0.001; visual mesh filename=/root/ibrido_ws/src/iit-centauro-ros-pkg/centauro_urdf/mesh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 scale=0.001 0.001 -0.001
- link wheel_4: geometry collision mesh filename=/root/ibrido_ws/src/iit-centauro-ros-pkg/centauro_urdf/mesh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 scale=0.001 0.001 0.001; visual mesh filename=/root/ibrido_ws/src/iit-centauro-ros-pkg/centauro_urdf/mesh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 scale=0.001 0.001 0.001
Joints:
- removed joint reference
- added joint floating_joint: type floating, parent world, child base_link, origin xyz=0.0 0.0 1.5

Commit message: added clock transmitter to allow using the -S option when running xbot2-core

File: tests/files/centauro.urdf (robot description, URDF)
Before this commit: robot centauro, 58 links, 57 joints
Joints:
- joint floating_joint: origin xyz=0.0 0.0 1.5 -> xyz=0.0 0.0 1.2

Commit message: MoveBaseNowTo working

File: tests/files/centauro.urdf (robot description, URDF)
Before this commit: robot centauro, 58 links, 57 joints
Joints:
- joint floating_joint: origin xyz=0.0 0.0 1.2 -> (none)

Commit message: using URDF with cylindrical wheels

File: tests/files/centauro.urdf (robot description, URDF)
Before this commit: robot centauro, 58 links, 57 joints
Links:
- link wheel_1: geometry collision cylinder length=0.03 radius=0.124; visual mesh filename=/root/ibrido_ws/src/iit-centauro-ros-pkg/centauro_urdf/mesh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 scale=0.001 0.001 -0.001
- link wheel_2: geometry collision cylinder length=0.03 radius=0.124; visual mesh filename=/root/ibrido_ws/src/iit-centauro-ros-pkg/centauro_urdf/mesh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 scale=0.001 0.001 0.001
- link wheel_3: geometry collision cylinder length=0.03 radius=0.124; visual mesh filename=/root/ibrido_ws/src/iit-centauro-ros-pkg/centauro_urdf/mesh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 scale=0.001 0.001 -0.001
- link wheel_4: geometry collision cylinder length=0.03 radius=0.124; visual mesh filename=/root/ibrido_ws/src/iit-centauro-ros-pkg/centauro_urdf/mesh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 scale=0.001 0.001 0.001
Joints:
- removed joint floating_joint
- added joint reference: type floating, parent world, child base_link
