Commit message: a bit of directory reorganization + added test files for unitree b2w

File: tests/files/centauro/centauro.urdf (robot description, URDF)
Before this commit: robot centauro, 58 links, 57 joints
Links:
- link D435_head_camera_link: geometry collision box size=0.02505 0.09 0.025

Commit message: removed .dae to allow mj to parse URDF

File: tests/files/centauro/centauro.urdf (robot description, URDF)
Before this commit: robot centauro, 58 links, 57 joints
Links:
- link D435i_camera_link: geometry collision box size=0.02505 0.09 0.025
